File: arduino/breakout/breakout.kicad_pcb (KiCad board)
At the start: 2 copper layers, 100 x 56 mm, 12 parts, among them SW1 PTS645SM43SMTR92 LFS, SW2 PTS645SM43SMTR92 LFS, SW3 PTS645SM43SMTR92 LFS, SW4 PTS645SM43SMTR92 LFS, SW5 PTS645SM43SMTR92 LFS, SW6 PTS645SM43SMTR92 LFS

Commit message: registry: every board rebuilt with pcbkit main 4684674e6 - the bought part named on the board
pcbkit dc07fdfd6 writes the bought row's MPN and Manufacturer (the design's own kept as DesignMPN /
DesignManufacturer) and the build chooses parts before it places (6361ec104). Each of the 44 boards
was rebuilt (; the two P4 boards  only: their builds reroute pairs):
copper unchanged on all 44 (segments, arcs and vias counted before and after), placement kept; the
Arduino and lab boards now carry the parts the catalogue gives them. The check gains only the new
judgements: part-maker (a part bought from another maker) and part-missing on hand-fitted modules
(DS1 sockets); p4-touch-7 loses part-stale. The P4 boards keep their hole-clearance errors (a
reroute is Team 3's).

Claude-Session: https://claude.ai/code/session_01BAgp959tApA8aEg85EYgfb
Parts:
- H1, H2, H3, H4: value (none) -> MountingHole_3.2mm_M3
Connections:
- SW1 pad 2: UP -> GND
- SW2 pad 2: DOWN -> GND
- SW3 pad 2: LEFT -> GND
- SW4 pad 2: RIGHT -> GND
- SW5 pad 2: A -> GND
- SW6 pad 2: B -> GND
