File: arduino/co2-monitor/co2-monitor.kicad_pcb (KiCad board)
At the start: 2 copper layers, 90 x 56 mm, 17 parts, among them U1 SCD40-D-R2

Commit message: boards: 15 boards rebuilt on pcbkit 20ffacdc9 (their pours under the 0.25 mm hole clearance)
Every board checked with main: 17 of 44 failed on hole-clearance (pours filled before fill c6 made
0.25 mm KiCad's hole clearance the default), keepout (holes now sized by the board) or
place-corner. design.run {} on each (placement and routing kept, pours refilled): 15 now complete,
0 errors. Not here: esp32-p4-touch-lcd-7b and p4-touch-7 (a build reroutes their pairs: 21 and 7
unrouted; kept as they were, 2,372 and 919 hole-clearance errors: a refill without a reroute is
needed).

Claude-Session: https://claude.ai/code/session_01BAgp959tApA8aEg85EYgfb
Parts:
- H1, H2, H3, H4: value (none) -> MountingHole_3.2mm_M3
Routing:
- net GND: track 1.54 -> 16.3 mm, vias 2 -> 6
- net SDA: track 121.3 -> 113.2 mm, vias 0 -> 1
- net V5: track 111.0 -> 115.5 mm, vias 1 -> 0
