File: arduino/egg-catcher/Egg-catcher.kicad_pcb (KiCad board)
At the start: 2 copper layers, 120 x 64 mm, 31 parts, among them J2 B2B-PH-K-S(LF)(SN), Q1 AO3401A, SW1 PTS645SM43SMTR92 LFS, SW2 PTS645SM43SMTR92 LFS, SW3 PTS645SM43SMTR92 LFS, SW4 PTS645SM43SMTR92 LFS, SW5 MSK12C02, U2 MCP73831T-2ACI/OT, U3 MT3608

Commit message: registry: every board rebuilt with pcbkit main 4684674e6 - the bought part named on the board
pcbkit dc07fdfd6 writes the bought row's MPN and Manufacturer (the design's own kept as DesignMPN /
DesignManufacturer) and the build chooses parts before it places (6361ec104). Each of the 44 boards
was rebuilt (; the two P4 boards  only: their builds reroute pairs):
copper unchanged on all 44 (segments, arcs and vias counted before and after), placement kept; the
Arduino and lab boards now carry the parts the catalogue gives them. The check gains only the new
judgements: part-maker (a part bought from another maker) and part-missing on hand-fitted modules
(DS1 sockets); p4-touch-7 loses part-stale. The P4 boards keep their hole-clearance errors (a
reroute is Team 3's).

Claude-Session: https://claude.ai/code/session_01BAgp959tApA8aEg85EYgfb
Parts:
- H1, H2, H3, H4: value (none) -> MountingHole_3.2mm_M3
- J1: value (none) -> USB4105-GF-A
Connections:
- SW1 pad 2: LEFT_UP -> GND
- SW2 pad 2: LEFT_DOWN -> GND
- SW3 pad 2: RIGHT_UP -> GND
- SW4 pad 2: RIGHT_DOWN -> GND
