File: arduino/simon/simon.kicad_pcb (KiCad board)
At the start: 2 copper layers, 80 x 80 mm, 16 parts, among them SW1 PTS645SM43SMTR92 LFS, SW2 PTS645SM43SMTR92 LFS, SW3 PTS645SM43SMTR92 LFS, SW4 PTS645SM43SMTR92 LFS

Commit message: Boards pass check and KiCad 10's DRC again: holes in courtyards, the USB net rename
pcbkit's check now has KiCad 10's pth/npth_inside_courtyard (pcbkit be5b6955), and 13 boards
failed it. KiCad's own DRC (kicad-cli 10) reports the same holes on every one of them.

- Parts that really stand above the holes under them (a screen or a Nano on its sockets, the
  Delta-S02's КМ-6 capacitors flat under its chips, as the factory placed them): a courtyard rule
  for the pair, written to each board's .kicad_dru, so KiCad's DRC agrees.
- Real collisions moved: servo-controller's dial 3 mm up (the Nano's socket pins came out under
  it), c3-pocket's fourth M3 hole from under a cell holder to the top edge's middle, s3-rgb's
  D-pad 2 mm up (a holder's peg came through under the down key).
- v003-emu, c3-pocket, rp2040-tft, rp2350-psram, s3-rgb, teensy41: re-routed for the standard USB
  block's renamed net (usb/raw is usb/vbusIn since pcbkit 2088839e): their tracks still carried
  the old name and shorted the fuse and connector pads.
- p4-touch-7: its board file still had a courtyard for the panel the design gives none (KiCad
  reported 114 courtyard errors); written again.

Measured on the dev host: all 44 registry boards `pcbkit check` complete with 0 errors, and
kicad-cli pcb drc 0 errors on every board.

Claude-Session: https://claude.ai/code/session_018URVYF1YPgyrMNetY9yT1T
Parts:
- H1, H2: value (none) -> MountingHole_3.2mm_M3

Commit message: registry: every board rebuilt with pcbkit main 4684674e6 - the bought part named on the board
pcbkit dc07fdfd6 writes the bought row's MPN and Manufacturer (the design's own kept as DesignMPN /
DesignManufacturer) and the build chooses parts before it places (6361ec104). Each of the 44 boards
was rebuilt (; the two P4 boards  only: their builds reroute pairs):
copper unchanged on all 44 (segments, arcs and vias counted before and after), placement kept; the
Arduino and lab boards now carry the parts the catalogue gives them. The check gains only the new
judgements: part-maker (a part bought from another maker) and part-missing on hand-fitted modules
(DS1 sockets); p4-touch-7 loses part-stale. The P4 boards keep their hole-clearance errors (a
reroute is Team 3's).

Claude-Session: https://claude.ai/code/session_01BAgp959tApA8aEg85EYgfb
Connections:
- SW1 pad 2: B1 -> GND
- SW2 pad 2: B2 -> GND
- SW3 pad 2: B3 -> GND
- SW4 pad 2: B4 -> GND
