File: arduino/thermostat/thermostat.kicad_pcb (KiCad board)
At the start: 2 copper layers, 90 x 56 mm, 16 parts, among them J1 RC servo header, 1 x 3 pins, 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, SW1 PTS645SM43SMTR92 LFS, SW2 PTS645SM43SMTR92 LFS, U1 SHT31-DIS-B2.5kS

Commit message: boards: 15 boards rebuilt on pcbkit 20ffacdc9 (their pours under the 0.25 mm hole clearance)
Every board checked with main: 17 of 44 failed on hole-clearance (pours filled before fill c6 made
0.25 mm KiCad's hole clearance the default), keepout (holes now sized by the board) or
place-corner. design.run {} on each (placement and routing kept, pours refilled): 15 now complete,
0 errors. Not here: esp32-p4-touch-lcd-7b and p4-touch-7 (a build reroutes their pairs: 21 and 7
unrouted; kept as they were, 2,372 and 919 hole-clearance errors: a refill without a reroute is
needed).

Claude-Session: https://claude.ai/code/session_01BAgp959tApA8aEg85EYgfb
Parts:
- H1, H2, H3, H4: value (none) -> MountingHole_3.2mm_M3
Connections:
- SW1 pad 2: MINUS -> GND
- SW2 pad 2: PLUS -> GND
