File: devices/can-node/can-node.kicad_pcb (KiCad board)
At the start: 2 copper layers, 60 x 40 mm, 68 parts, among them J1 SM04B-GHS-TB, Q1 AO3401A, U1 STM32G431CBU6, U2 SN65HVD230DR, U3 ICM-42688-P, U4 TPS54331D, Y1 8MHz 10pF

Commit message: registry: every board rebuilt with pcbkit main 4684674e6 - the bought part named on the board
pcbkit dc07fdfd6 writes the bought row's MPN and Manufacturer (the design's own kept as DesignMPN /
DesignManufacturer) and the build chooses parts before it places (6361ec104). Each of the 44 boards
was rebuilt (; the two P4 boards  only: their builds reroute pairs):
copper unchanged on all 44 (segments, arcs and vias counted before and after), placement kept; the
Arduino and lab boards now carry the parts the catalogue gives them. The check gains only the new
judgements: part-maker (a part bought from another maker) and part-missing on hand-fitted modules
(DS1 sockets); p4-touch-7 loses part-stale. The P4 boards keep their hole-clearance errors (a
reroute is Team 3's).

Claude-Session: https://claude.ai/code/session_01BAgp959tApA8aEg85EYgfb
Parts:
- H1, H2: value (none) -> MountingHole_2.7mm_M2.5_Pad; footprint MountingHole_3.2mm_M3_Pad -> MountingHole_2.7mm_M2.5_Pad
- J2: value (none) -> PinHeader_1x02_P2.54mm_Vertical
- J3: value (none) -> PinHeader_1x03_P2.54mm_Vertical
- J4: value (none) -> PinHeader_1x05_P2.54mm_Vertical
- J5: value (none) -> PinHeader_2x04_P2.54mm_Vertical
