File: devices/esp32-p4-touch-lcd-7b/esp32-p4-touch-lcd-7b.kicad_pcb (KiCad board)
At the start: 6 copper layers, 165.5 x 98 mm, 334 parts, among them J1 USB-A 90deg, J2 FPC 1.0mm 15P flip-lock botto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, J3 FPC 0.5mm 6P flip-lock top co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, J4 PH2.0-2P SMD vertical, J5 USB4105-GF-A, J6 USB4105-GF-A, M1 NDC7002N, P1 PH2.0-12P SMD vertical, P2 FPC 0.5mm 30P flip-lock botto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, P3 PH2.0-12P SMD vertical, Q1 AO3401A, Q2 AO3401A, Q3 AO3401A, Q5 AO3401A, Q6 AO3401A, Q8 AO3401A, Q9 MMBT3904-7-F, SW1 PTS645SM43SMTR92 LFS, SW2 MSK12C02, U1 ESP32-C6-MINI-1-N4, U10 RT9193-18GB, U11 SP3485EN-L/TR, U12 AP3032KTR-G1, U13 ESP32-P4NRW32, U14 TJA1051T/3/1J, U15 RT9193-33GB, U16 ES8311, U17 ES7210, U18 MMDT3906DW, U19 NS4150B, U2 SY6280AAC, U20 IP5306, U21 GD25Q256EYIGR, U23 MMDT3906DW, U24 MMDT3906DW, U3 SY8089AAAC, U4 MMDT3906DW, U5 SY8089AAAC, U6 CH343P, U7 USBLC6-2SC6, U7A MMBT3904-7-F, U7B MMBT3904-7-F, U8 USBLC6-2SC6, U9 AP3012KTR-E1, Y1 40MHz 10pF, Y3 Q13FC13500004

Commit message: lab, examples, esp32-p4-touch-lcd-7b: the sweep's errors and stale parts
- lab/stopwatch: the display module stands on its socket above the Nano's socket pins. It now has
  the courtyard waiver the other Nano boards have (13 pth-inside-courtyard -> 0).
- lab/servo-controller: outline 90 x 80 -> 70 x 70 mm, with the parts where they were
  (board-oversized, plan-size: 11 % parts). Complete, 0 warnings.
- examples/blinker, examples/led-bar, devices/esp32-p4-touch-lcd-7b: `pcbkit parts` chose again
  where the recorded part no longer met the need (part-stale).

Claude-Session: https://claude.ai/code/session_01B3VRfBCg9vAvGVWujVGarr
Parts:
- removed the LCD1 at (182.8, 151.0) (x42)
- added LCD1: touch-display, Waveshare-7inch-1024x600-DSI, B.Cu at (182.8, 151.0)
- LSK1, LSK2, LSK3, LSK4: value (none) -> MountingHole_2.7mm_M2.5
Connections:
- Key1 pad 2: ESP_EN -> GND
- Key2 pad 2: BOOT -> GND
- SW1 pad 2: Net-(SW1-1) -> GND

Commit message: devices/esp32-p4-touch-lcd-7b: its pours refilled under the 0.25 mm hole clearance (design.run { only: fill })
Main (d5fe8dd89) checked it with 2,372 hole-clearance and 2 pour-stale errors: its pours were
filled before fill c6. A refill alone (no reroute) takes it to 1,213 hole-clearance errors, 0
unrouted. Left: routed tracks and vias closer than 0.25 mm to via drills, laid before the rule; a
build reroutes and leaves nets unrouted (team 3). p4-touch-7 not here: a refill splits its VSYS pour.

Claude-Session: https://claude.ai/code/session_01BAgp959tApA8aEg85EYgfb
Parts:
- L5, L7, R38, R_MIC1, R_MIC2, R_VCC: value 0mohm -> 0uohm
