File: doom/f411-psram/doom-05-f411-psram.kicad_pcb (KiCad board)
At the start: 4 copper layers, 140 x 104 mm, 79 parts, among them J5 S2B-PH-K-S(LF)(SN), Q1 AO3401A, Q2 FS8205A, SW1 PTS645SM43SMTR92 LFS, SW10 TS-1187A-B-A-B, SW11 TS-1187A-B-A-B, SW2 PTS645SM43SMTR92 LFS, SW3 PTS645SM43SMTR92 LFS, SW4 PTS645SM43SMTR92 LFS, SW5 PTS645SM43SMTR92 LFS, SW6 PTS645SM43SMTR92 LFS, SW7 PTS645SM43SMTR92 LFS, SW8 PTS645SM43SMTR92 LFS, SW9 MSK12C02, U1 STM32F411CEU6, U2 APS6404L-3SQR-SN, U3 W25Q128JVSIQ, U4 TLV75533PDBVR, U5 MAX98357AETE+T, U6 BQ24075RGTR, U7 DW01A, U8 ESD 2-line, Y1 25MHz 10pF

Commit message: doom, examples: re-route around the USB-C receptacle's new land pattern
The standard receptacle became GCT USB4105's recommended layout (pcbkit 7e43c086): its shield
legs moved and two unplated guide holes appeared, under the copper these boards had been routed
with (solder-mask-bridge and clearance errors at J1). `build.run` re-routed the 3–5 nets that
crossed it: all seven check complete with 0 errors again; the six Doom boards export for the fab
without --force.

Claude-Session: https://claude.ai/code/session_01GffCzZXi9ShujPbky1eccg
Parts:
- J2: value (none) -> USB4105-GF-A
- U8: value ESD 2-line -> USBLC6-2SC6
Routing:
- net DN: track 66.4 -> 47.5 mm, vias 6 -> 1
- net DP: track 65.6 -> 52.0 mm, vias 4 -> 2
- net VBUS: track 87.2 -> 88.4 mm

Commit message: doom: a resettable fuse per 18650 cell, a 2 % backlight clamp, a 1 A LDO on the S3 boards
The verifier (wiring-parallel-cells) found the two holders of every Doom board directly in parallel:
a cell put in backwards, or one much fuller than the other, drives the other through nothing but
the cells' resistance (about 56-168 A). Each holder's + now reaches BAT_IN through its own 2 A
resettable fuse (Littelfuse 1812L200/16GR, C18198340: 16 V, 100 A interrupting) on new nets
CELL1_P / CELL2_P. Nothing else moved; the boards were re-routed for the new nets.

- s3-rgb: the MT3608 backlight's open-panel clamp was a 28 V 5 % zener (bound 30.0 V against the
  switch's 30 V). It is now two 2 % zeners in series, UDZVTE-1718B + UDZVTE-1710B (27.33-28.56 V;
  LCSC stocks no single 28 V 2 % part). That is under 29.2 V and above the panel's 27.2 V.
- s3-rgb, s3-handheld: TLV75533 (500 mA) -> TLV75733 (1 A, C485517, same DBV pins; sheet from
  SBVS322C), for the ESP32-S3's 500 mA supply peaks (erc-supply-peak).
- c3-pocket, v003-emu: the USB PTC's hold is 750 mA, as the part (nSMD075) is (rating-current).
- pico2-carrier: the CHG/PG LEDs 1.5 mm further from the display's courtyard. rp2350-handheld:
  the logo off the LCD's courtyard and BT1's peg.
- READMEs: the per-cell fuses, the boards already ordered (s3-rgb, JLC W2026102705013253: insert
  the cells one at a time), status and BOM as check and the fab export give them now.

Measured on the dev host (pcbkit 5e0d2cc8): all 11 complete, 0 errors, 0 unrouted. What is left is
erc-rail-name (sent to the verifier as false positives) and full-speed USB pair coupling. The MCU
pins' nets are unchanged on every board, so the firmware and its simulation are unchanged.

Claude-Session: https://claude.ai/code/session_01B3VRfBCg9vAvGVWujVGarr
Parts:
- added F1: PTC 2000mA, Fuse_1812_4532Metric, B.Cu at (124.8, 191.8)
- added F2: PTC 2000mA, Fuse_1812_4532Metric, B.Cu at (124.8, 169.8)
- H1, H2, H3, H4: value (none) -> MountingHole_3.2mm_M3
- J1: value (none) -> PinHeader_1x05_P2.54mm_Vertical
- logo: value (none) -> Logo_PCBKit_pcbkit.io
- tpBat, tpGnd, tpSys, tpV3: value (none) -> TestPoint_Round_D1.5mm
Connections:
- BT1 pad 2: BAT_IN -> CELL1_P
- BT2 pad 2: BAT_IN -> CELL2_P
- SW1 pad 2: UP -> GND
- SW10 pad 2: BOOT0 -> V3
- SW11 pad 2: NRST -> GND
- SW2 pad 2: DOWN -> GND
- SW3 pad 2: LEFT -> GND
- SW4 pad 2: RIGHT -> GND
- SW5 pad 2: FIRE -> GND
- SW6 pad 2: USE -> GND
- SW7 pad 2: STRAFE -> GND
- SW8 pad 2: MENU -> GND
Routing:
- net BAT_IN: track 47.3 -> 56.9 mm
- net CELL2_P: track 0.00 -> 6.98 mm
- net CELL1_P: track 0.00 -> 6.98 mm
- net V3: track 214.0 -> 209.5 mm
- net MEM_MOSI: track 35.8 -> 33.5 mm
- net FIRE: track 64.6 -> 63.2 mm
- net Net-(C19-1): track 5.42 -> 4.06 mm
- net NRST: track 84.3 -> 83.5 mm
- net VBUS: track 88.4 -> 87.7 mm
