File: doom/s3-handheld/doom-08-s3-handheld.kicad_pcb (KiCad board)
At the start: 4 copper layers, 156 x 110 mm, 75 parts, among them J4 DM3AT-SF-PEJM5, J5 S2B-PH-K-S(LF)(SN), Q1 AO3401A, Q2 FS8205A, SW1 PTS645SM43SMTR92 LFS, SW10 PTS645SM43SMTR92 LFS, SW11 TS-1187A-B-A-B, SW12 MSK12C02, SW2 PTS645SM43SMTR92 LFS, SW3 PTS645SM43SMTR92 LFS, SW4 PTS645SM43SMTR92 LFS, SW5 PTS645SM43SMTR92 LFS, SW6 PTS645SM43SMTR92 LFS, SW7 PTS645SM43SMTR92 LFS, SW8 PTS645SM43SMTR92 LFS, SW9 PTS645SM43SMTR92 LFS, U1 ESP32-S3-WROOM-1-N16R8, U2 ESD 2-line, U4 TLV75533PDBVR, U5 MAX98357AETE+T, U6 BQ24075RGTR, U7 MAX17048G+T10, U8 DW01A

Commit message: doom, examples: re-route around the USB-C receptacle's new land pattern
The standard receptacle became GCT USB4105's recommended layout (pcbkit 7e43c086): its shield
legs moved and two unplated guide holes appeared, under the copper these boards had been routed
with (solder-mask-bridge and clearance errors at J1). `build.run` re-routed the 3–5 nets that
crossed it: all seven check complete with 0 errors again; the six Doom boards export for the fab
without --force.

Claude-Session: https://claude.ai/code/session_01GffCzZXi9ShujPbky1eccg
Parts:
- J1: value (none) -> USB4105-GF-A
- U2: value ESD 2-line -> USBLC6-2SC6
Routing:
- net DP: track 96.5 -> 39.2 mm, vias 6 -> 2
- net DN: track 58.0 -> 39.5 mm, vias 4 -> 2
- net VBUS: track 86.4 -> 88.5 mm, vias 6 -> 5
- net GND: vias 3 -> 4

Commit message: Boards pass check and KiCad 10's DRC again: holes in courtyards, the USB net rename
pcbkit's check now has KiCad 10's pth/npth_inside_courtyard (pcbkit be5b6955), and 13 boards
failed it. KiCad's own DRC (kicad-cli 10) reports the same holes on every one of them.

- Parts that really stand above the holes under them (a screen or a Nano on its sockets, the
  Delta-S02's КМ-6 capacitors flat under its chips, as the factory placed them): a courtyard rule
  for the pair, written to each board's .kicad_dru, so KiCad's DRC agrees.
- Real collisions moved: servo-controller's dial 3 mm up (the Nano's socket pins came out under
  it), c3-pocket's fourth M3 hole from under a cell holder to the top edge's middle, s3-rgb's
  D-pad 2 mm up (a holder's peg came through under the down key).
- v003-emu, c3-pocket, rp2040-tft, rp2350-psram, s3-rgb, teensy41: re-routed for the standard USB
  block's renamed net (usb/raw is usb/vbusIn since pcbkit 2088839e): their tracks still carried
  the old name and shorted the fuse and connector pads.
- p4-touch-7: its board file still had a courtyard for the panel the design gives none (KiCad
  reported 114 courtyard errors); written again.

Measured on the dev host: all 44 registry boards `pcbkit check` complete with 0 errors, and
kicad-cli pcb drc 0 errors on every board.

Claude-Session: https://claude.ai/code/session_018URVYF1YPgyrMNetY9yT1T
Parts:
- H1, H2, H3, H4: value (none) -> MountingHole_3.2mm_M3
- logo: value (none) -> Logo_PCBKit_pcbkit.io
- tpBat, tpGnd, tpSys, tpV3: value (none) -> TestPoint_Round_D1.5mm
Routing:
- net BAT_IN: track 55.6 -> 32.2 mm
- net TS: track 9.57 -> 7.72 mm
- net Net-(Q2-5): track 15.9 -> 14.3 mm
- net SD_D1: track 4.75 -> 3.57 mm
- net I2S_DIN: track 77.0 -> 76.0 mm
- net Net-(C8-1): track 6.08 -> 5.21 mm
- net CHG_N: track 15.2 -> 14.4 mm
- net EN: track 86.9 -> 86.1 mm
- net SD_D3: track 7.42 -> 6.71 mm
- net usb/power/cc1: track 5.27 -> 4.62 mm
- net BAT: track 107.2 -> 106.6 mm

Commit message: doom: a resettable fuse per 18650 cell, a 2 % backlight clamp, a 1 A LDO on the S3 boards
The verifier (wiring-parallel-cells) found the two holders of every Doom board directly in parallel:
a cell put in backwards, or one much fuller than the other, drives the other through nothing but
the cells' resistance (about 56-168 A). Each holder's + now reaches BAT_IN through its own 2 A
resettable fuse (Littelfuse 1812L200/16GR, C18198340: 16 V, 100 A interrupting) on new nets
CELL1_P / CELL2_P. Nothing else moved; the boards were re-routed for the new nets.

- s3-rgb: the MT3608 backlight's open-panel clamp was a 28 V 5 % zener (bound 30.0 V against the
  switch's 30 V). It is now two 2 % zeners in series, UDZVTE-1718B + UDZVTE-1710B (27.33-28.56 V;
  LCSC stocks no single 28 V 2 % part). That is under 29.2 V and above the panel's 27.2 V.
- s3-rgb, s3-handheld: TLV75533 (500 mA) -> TLV75733 (1 A, C485517, same DBV pins; sheet from
  SBVS322C), for the ESP32-S3's 500 mA supply peaks (erc-supply-peak).
- c3-pocket, v003-emu: the USB PTC's hold is 750 mA, as the part (nSMD075) is (rating-current).
- pico2-carrier: the CHG/PG LEDs 1.5 mm further from the display's courtyard. rp2350-handheld:
  the logo off the LCD's courtyard and BT1's peg.
- READMEs: the per-cell fuses, the boards already ordered (s3-rgb, JLC W2026102705013253: insert
  the cells one at a time), status and BOM as check and the fab export give them now.

Measured on the dev host (pcbkit 5e0d2cc8): all 11 complete, 0 errors, 0 unrouted. What is left is
erc-rail-name (sent to the verifier as false positives) and full-speed USB pair coupling. The MCU
pins' nets are unchanged on every board, so the firmware and its simulation are unchanged.

Claude-Session: https://claude.ai/code/session_01B3VRfBCg9vAvGVWujVGarr
Parts:
- added F1: PTC 2000mA, Fuse_1812_4532Metric, B.Cu at (157.5, 182.5)
- added F2: PTC 2000mA, Fuse_1812_4532Metric, B.Cu at (158.8, 169.8)
- U4: value TLV75533PDBVR -> TLV75733PDBVR
Connections:
- BT1 pad 2: BAT_IN -> CELL1_P
- BT2 pad 2: BAT_IN -> CELL2_P
- SW1 pad 2: UP -> GND
- SW10 pad 2: ENTER -> GND
- SW11 pad 2: EN -> GND
- SW2 pad 2: DOWN -> GND
- SW3 pad 2: LEFT -> GND
- SW4 pad 2: RIGHT -> GND
- SW5 pad 2: STRAFE_L -> GND
- SW6 pad 2: STRAFE_R -> GND
- SW7 pad 2: FIRE -> GND
- SW8 pad 2: USE -> GND
- SW9 pad 2: MENU -> GND
Routing:
- net BAT_IN: track 32.2 -> 9.88 mm
- net CELL1_P: track 0.00 -> 8.13 mm
- net CELL2_P: track 0.00 -> 6.98 mm
- net usb/power/cc1: track 4.62 -> 3.97 mm

Commit message: boards: 15 boards rebuilt on pcbkit 20ffacdc9 (their pours under the 0.25 mm hole clearance)
Every board checked with main: 17 of 44 failed on hole-clearance (pours filled before fill c6 made
0.25 mm KiCad's hole clearance the default), keepout (holes now sized by the board) or
place-corner. design.run {} on each (placement and routing kept, pours refilled): 15 now complete,
0 errors. Not here: esp32-p4-touch-lcd-7b and p4-touch-7 (a build reroutes their pairs: 21 and 7
unrouted; kept as they were, 2,372 and 919 hole-clearance errors: a refill without a reroute is
needed).

Claude-Session: https://claude.ai/code/session_01BAgp959tApA8aEg85EYgfb
Routing:
- net DP: track 38.8 -> 69.5 mm, vias 2 -> 4
