File: examples/blinker/board.kicad_pcb (KiCad board)
At the start: 2 copper layers, 27 x 23 mm, 12 parts

Commit message: p4-touch-7, blinker, led-bar: parts chosen from JLCPCB's catalogue, the fab files export
Since the parts selection buys from JLCPCB's own catalogue, these boards' support capacitors and
connectors had no orderable part and export.run refused them. parts.select chose every group
(p4-touch-7's 40 MHz crystal pinned as on the 7B board, C426988); copper unchanged.

Claude-Session: https://claude.ai/code/session_01GffCzZXi9ShujPbky1eccg
Parts:
- U1: value (none) -> NE555DR

Commit message: lab, examples, esp32-p4-touch-lcd-7b: the sweep's errors and stale parts
- lab/stopwatch: the display module stands on its socket above the Nano's socket pins. It now has
  the courtyard waiver the other Nano boards have (13 pth-inside-courtyard -> 0).
- lab/servo-controller: outline 90 x 80 -> 70 x 70 mm, with the parts where they were
  (board-oversized, plan-size: 11 % parts). Complete, 0 warnings.
- examples/blinker, examples/led-bar, devices/esp32-p4-touch-lcd-7b: `pcbkit parts` chose again
  where the recorded part no longer met the need (part-stale).

Claude-Session: https://claude.ai/code/session_01B3VRfBCg9vAvGVWujVGarr
Parts:
- D1: value (none) -> LED_0603_1608Metric
- H1, H2, H3, H4: value (none) -> MountingHole_3.2mm_M3_Pad
- J1: value (none) -> PinHeader_1x02_P2.54mm_Vertical
Changed lines of the file:
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@@
     (property "pcbkit" "C1" (at 0 0 0) (layer "F.Fab") (hide yes) (effects (font (size 1 1))))
     (property "pcbkit-need" "a8c907816db1 MPN Manufacturer" (at 0 0 0) (layer "F.Fab") (hide yes) (effects (font (size 1 1))))
-    (duplicate_pad_numbers_are_jumpers no)
     (fp_rect (start -1.7 0.98) (end 1.7 -0.98) (stroke (width 0.05) (type solid)) (layer "F.CrtYd"))
     (fp_line (start -0.19 0.735) (end 0.19 0.735) (stroke (width 0.12) (type solid)) (layer "F.SilkS"))
@@
     (property "Manufacturer" "YAGEO" (at 0 0 0) (layer "F.Fab") (hide yes) (effects (font (size 1 1))))
     (property "pcbkit" "C2" (at 0 0 0) (layer "F.Fab") (hide yes) (effects (font (size 1 1))))
-    (property "pcbkit-need" "9211953334ff MPN Manufacturer" (at 0 0 0) (layer "F.Fab") (hide yes) (effects (font (size 1 1))))
-    (duplicate_pad_numbers_are_jumpers no)
+    (property "pcbkit-need" "8b728515c591 MPN Manufacturer" (at 0 0 0) (layer "F.Fab") (hide yes) (effects (font (size 1 1))))
     (fp_rect (start -1.48 0.73) (end 1.48 -0.73) (stroke (width 0.05) (type solid)) (layer "F.CrtYd"))
     (pad "1" smd roundrect (at -0.775 0 180) (size 0.9 0.95) (layers "F.Cu" "F.Paste" "F.Mask") (roundrect_rratio 0.250000000000) (solder_mask_margin 0.05) (net 6 "VCC"))
@@
     (tags "chip 0603 1608Metric")
     (property "Reference" "D1" (at 0 -1.43 0) (layer "F.SilkS") (effects (font (size 1 1) (thickness 0.15))))
-    (property "Value" "" (at 0 0 0) (layer "F.Fab") (hide yes) (effects (font (size 1 1))))
+    (property "Value" "LED_0603_1608Metric" (at 0 0 0) (layer "F.Fab") (hide yes) (effects (font (size 1 1))))
     (property "LCSC Part #" "C2286" (at 0 0 0) (layer "F.Fab") (hide yes) (effects (font (size 1 1))))
     (property "MPN" "KT-0603R" (at 0 0 0) (layer "F.Fab") (hide yes) (effects (font (size 1 1))))
@@
     (property "pcbkit" "D1" (at 0 0 0) (layer "F.Fab") (hide yes) (effects (font (size 1 1))))
     (property "pcbkit-need" "0e3735e21846 MPN Manufacturer" (at 0 0 0) (layer "F.Fab") (hide yes) (effects (font (size 1 1))))
-    (duplicate_pad_numbers_are_jumpers no)
     (fp_rect (start -1.48 0.73) (end 1.48 -0.73) (stroke (width 0.05) (type solid)) (layer "F.CrtYd"))
     (fp_line (start 0.8 -0.735) (end -1.485 -0.735) (stroke (width 0.12) (type solid)) (layer "F.SilkS"))
@@
     (tags "mounting hole M3")
     (property "Reference" "H1" (at 0 0 0) (layer "F.Fab") (hide yes) (effects (font (size 1 1))))
-    (property "Value" "" (at 0 0 0) (layer "F.Fab") (hide yes) (effects (font (size 1 1))))
+    (property "Value" "MountingHole_3.2mm_M3_Pad" (at 0 0 0) (layer "F.Fab") (hide yes) (effects (font (size 1 1))))
     (property "pcbkit" "holes/holes[0]" (at 0 0 0) (layer "F.Fab") (hide yes) (effects (font (size 1 1))))
-    (duplicate_pad_numbers_are_jumpers no)
     (fp_rect (start -3.45 3.45) (end 3.45 -3.45) (stroke (width 0.05) (type solid)) (layer "F.CrtYd"))
     (pad "1" thru_hole circle (at 0 0 0) (size 6.4 6.4) (drill 3.2) (layers "*.Cu" "*.Mask") (solder_mask_margin 0.05))
@@
     (tags "mounting hole M3")
     (property "Reference" "H2" (at 0 0 0) (layer "F.Fab") (hide yes) (effects (font (size 1 1))))
-    (property "Value" "" (at 0 0 0) (layer "F.Fab") (hide yes) (effects (font (size 1 1))))
+    (property "Value" "MountingHole_3.2mm_M3_Pad" (at 0 0 0) (layer "F.Fab") (hide yes) (effects (font (size 1 1))))
     (property "pcbkit" "holes/holes[1]" (at 0 0 0) (layer "F.Fab") (hide yes) (effects (font (size 1 1))))
-    (duplicate_pad_numbers_are_jumpers no)
     (fp_rect (start -3.45 3.45) (end 3.45 -3.45) (stroke (width 0.05) (type solid)) (layer "F.CrtYd"))
     (pad "1" thru_hole circle (at 0 0 0) (size 6.4 6.4) (drill 3.2) (layers "*.Cu" "*.Mask") (solder_mask_margin 0.05))
@@
     (tags "mounting hole M3")
     (property "Reference" "H3" (at 0 0 0) (layer "F.Fab") (hide yes) (effects (font (size 1 1))))
-    (property "Value" "" (at 0 0 0) (layer "F.Fab") (hide yes) (effects (font (size 1 1))))
+    (property "Value" "MountingHole_3.2mm_M3_Pad" (at 0 0 0) (layer "F.Fab") (hide yes) (effects (font (size 1 1))))
     (property "pcbkit" "holes/holes[2]" (at 0 0 0) (layer "F.Fab") (hide yes) (effects (font (size 1 1))))
-    (duplicate_pad_numbers_are_jumpers no)
     (fp_rect (start -3.45 3.45) (end 3.45 -3.45) (stroke (width 0.05) (type solid)) (layer "F.CrtYd"))
     (pad "1" thru_hole circle (at 0 0 0) (size 6.4 6.4) (drill 3.2) (layers "*.Cu" "*.Mask") (solder_mask_margin 0.05))
@@
     (tags "mounting hole M3")
     (property "Reference" "H4" (at 0 0 0) (layer "F.Fab") (hide yes) (effects (font (size 1 1))))
-    (property "Value" "" (at 0 0 0) (layer "F.Fab") (hide yes) (effects (font (size 1 1))))
+    (property "Value" "MountingHole_3.2mm_M3_Pad" (at 0 0 0) (layer "F.Fab") (hide yes) (effects (font (size 1 1))))
     (property "pcbkit" "holes/holes[3]" (at 0 0 0) (layer "F.Fab") (hide yes) (effects (font (size 1 1))))
-    (duplicate_pad_numbers_are_jumpers no)
     (fp_rect (start -3.45 3.45) (end 3.45 -3.45) (stroke (width 0.05) (type solid)) (layer "F.CrtYd"))
     (pad "1" thru_hole circle (at 0 0 0) (size 6.4 6.4) (drill 3.2) (layers "*.Cu" "*.Mask") (solder_mask_margin 0.05))
@@
     (tags "THT pin header")
     (property "Reference" "J1" (at 0 -3.49 180) (layer "F.SilkS") (effects (font (size 1 1) (thickness 0.15))))
-    (property "Value" "" (at 0 0 0) (layer "F.Fab") (hide yes) (effects (font (size 1 1))))
+    (property "Value" "PinHeader_1x02_P2.54mm_Vertical" (at 0 0 0) (layer "F.Fab") (hide yes) (effects (font (size 1 1))))
     (property "LCSC Part #" "C358684" (at 0 0 0) (layer "F.Fab") (hide yes) (effects (font (size 1 1))))
     (property "MPN" "MTP125-1102S1" (at 0 0 0) (layer "F.Fab") (hide yes) (effects (font (size 1 1))))
@@
     (property "pcbkit" "J1" (at 0 0 0) (layer "F.Fab") (hide yes) (effects (font (size 1 1))))
     (property "pcbkit-need" "e89ca4e0fa5d MPN Manufacturer" (at 0 0 0) (layer "F.Fab") (hide yes) (effects (font (size 1 1))))
-    (duplicate_pad_numbers_are_jumpers no)
     (fp_rect (start -1.52 2.79) (end 1.52 -2.79) (stroke (width 0.05) (type solid)) (layer "F.CrtYd"))
     (fp_line (start 0 -2.65) (end -1.38 -2.65) (stroke (width 0.12) (type solid)) (layer "F.SilkS"))
@@
     (property "pcbkit" "R1" (at 0 0 0) (layer "F.Fab") (hide yes) (effects (font (size 1 1))))
     (property "pcbkit-need" "02d78dfd10f6 MPN Manufacturer" (at 0 0 0) (layer "F.Fab") (hide yes) (effects (font (size 1 1))))
-    (duplicate_pad_numbers_are_jumpers no)
     (fp_rect (start -1.48 0.73) (end 1.48 -0.73) (stroke (width 0.05) (type solid)) (layer "F.CrtYd"))
     (fp_line (start -0.165 0.5225) (end 0.165 0.5225) (stroke (width 0.12) (type solid)) (layer "F.SilkS"))
@@
     (property "pcbkit" "R2" (at 0 0 0) (layer "F.Fab") (hide yes) (effects (font (size 1 1))))
     (property "pcbkit-need" "dcccc1ed6988 MPN Manufacturer" (at 0 0 0) (layer "F.Fab") (hide yes) (effects (font (size 1 1))))
-    (duplicate_pad_numbers_are_jumpers no)
     (fp_rect (start -1.48 0.73) (end 1.48 -0.73) (stroke (width 0.05) (type solid)) (layer "F.CrtYd"))
     (fp_line (start -0.165 0.5225) (end 0.165 0.5225) (stroke (width 0.12) (type solid)) (layer "F.SilkS"))
@@
     (property "pcbkit" "R3" (at 0 0 0) (layer "F.Fab") (hide yes) (effects (font (size 1 1))))
     (property "pcbkit-need" "c037995ebaed MPN Manufacturer" (at 0 0 0) (layer "F.Fab") (hide yes) (effects (font (size 1 1))))
-    (duplicate_pad_numbers_are_jumpers no)
     (fp_rect (start -1.48 0.73) (end 1.48 -0.73) (stroke (width 0.05) (type solid)) (layer "F.CrtYd"))
     (fp_line (start -0.165 0.5225) (end 0.165 0.5225) (stroke (width 0.12) (type solid)) (layer "F.SilkS"))
@@
     (property "pcbkit" "U1" (at 0 0 0) (layer "F.Fab") (hide yes) (effects (font (size 1 1))))
     (property "pcbkit-need" "0042c0ac09cd" (at 0 0 0) (layer "F.Fab") (hide yes) (effects (font (size 1 1))))
-    (duplicate_pad_numbers_are_jumpers no)
     (fp_rect (start -3.7 2.7) (end 3.7 -2.7) (stroke (width 0.05) (type solid)) (layer "F.CrtYd"))
     (fp_line (start -2.06 2.465) (end -2.06 2.56) (stroke (width 0.12) (type solid)) (layer "F.SilkS"))

Commit message: boards: 15 boards rebuilt on pcbkit 20ffacdc9 (their pours under the 0.25 mm hole clearance)
Every board checked with main: 17 of 44 failed on hole-clearance (pours filled before fill c6 made
0.25 mm KiCad's hole clearance the default), keepout (holes now sized by the board) or
place-corner. design.run {} on each (placement and routing kept, pours refilled): 15 now complete,
0 errors. Not here: esp32-p4-touch-lcd-7b and p4-touch-7 (a build reroutes their pairs: 21 and 7
unrouted; kept as they were, 2,372 and 919 hole-clearance errors: a refill without a reroute is
needed).

Claude-Session: https://claude.ai/code/session_01BAgp959tApA8aEg85EYgfb
Parts:
- H1, H2, H3, H4: value MountingHole_3.2mm_M3_Pad -> MountingHole_2.2mm_M2_Pad; footprint MountingHole_3.2mm_M3_Pad -> MountingHole_2.2mm_M2_Pad
- moved H1 1.41 mm to (102.7, 197.3)
- moved H2 1.41 mm to (124.3, 197.3)
- moved H3 1.41 mm to (124.3, 179.7)
- moved H4 1.41 mm to (102.7, 179.7)
Changed lines of the file:
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@@
     (descr "Multilayer ceramic capacitor 0603 (1608 metric), IPC-7351B nominal density")
     (tags "chip 0603 1608Metric")
-    (property "Reference" "C2" (at 0 -1.43 180) (layer "F.SilkS") (effects (font (size 1 1) (thickness 0.15))))
+    (property "Reference" "C2" (at 0 -1.455 180) (layer "F.SilkS") (effects (font (size 1 1) (thickness 0.15))))
     (property "Value" "100nF" (at 0 0 0) (layer "F.Fab") (hide yes) (effects (font (size 1 1))))
     (property "LCSC Part #" "C14663" (at 0 0 0) (layer "F.Fab") (hide yes) (effects (font (size 1 1))))
@@
     (pad "2" smd roundrect (at 0.7875 0 0) (size 0.875 0.95) (layers "F.Cu" "F.Paste" "F.Mask") (roundrect_rratio 0.250000000000) (solder_mask_margin 0.05) (net 3 "LEDK"))
   )
-  (footprint "MountingHole_3.2mm_M3_Pad" (layer "F.Cu") (at 103.743 196.257 0)
-    (descr "Mounting hole for M3, plated")
-    (tags "mounting hole M3")
+  (footprint "MountingHole_2.2mm_M2_Pad" (layer "F.Cu") (at 102.743 197.257 0)
+    (descr "Mounting hole for M2, plated")
+    (tags "mounting hole M2")
     (property "Reference" "H1" (at 0 0 0) (layer "F.Fab") (hide yes) (effects (font (size 1 1))))
-    (property "Value" "MountingHole_3.2mm_M3_Pad" (at 0 0 0) (layer "F.Fab") (hide yes) (effects (font (size 1 1))))
+    (property "Value" "MountingHole_2.2mm_M2_Pad" (at 0 0 0) (layer "F.Fab") (hide yes) (effects (font (size 1 1))))
     (property "pcbkit" "holes/holes[0]" (at 0 0 0) (layer "F.Fab") (hide yes) (effects (font (size 1 1))))
-    (fp_rect (start -3.45 3.45) (end 3.45 -3.45) (stroke (width 0.05) (type solid)) (layer "F.CrtYd"))
-    (pad "1" thru_hole circle (at 0 0 0) (size 6.4 6.4) (drill 3.2) (layers "*.Cu" "*.Mask") (solder_mask_margin 0.05))
+    (fp_rect (start -2.45 2.45) (end 2.45 -2.45) (stroke (width 0.05) (type solid)) (layer "F.CrtYd"))
+    (pad "1" thru_hole circle (at 0 0 0) (size 4.4 4.4) (drill 2.2) (layers "*.Cu" "*.Mask") (solder_mask_margin 0.05))
   )
-  (footprint "MountingHole_3.2mm_M3_Pad" (layer "F.Cu") (at 123.257 196.257 0)
-    (descr "Mounting hole for M3, plated")
-    (tags "mounting hole M3")
+  (footprint "MountingHole_2.2mm_M2_Pad" (layer "F.Cu") (at 124.257 197.257 0)
+    (descr "Mounting hole for M2, plated")
+    (tags "mounting hole M2")
     (property "Reference" "H2" (at 0 0 0) (layer "F.Fab") (hide yes) (effects (font (size 1 1))))
-    (property "Value" "MountingHole_3.2mm_M3_Pad" (at 0 0 0) (layer "F.Fab") (hide yes) (effects (font (size 1 1))))
+    (property "Value" "MountingHole_2.2mm_M2_Pad" (at 0 0 0) (layer "F.Fab") (hide yes) (effects (font (size 1 1))))
     (property "pcbkit" "holes/holes[1]" (at 0 0 0) (layer "F.Fab") (hide yes) (effects (font (size 1 1))))
-    (fp_rect (start -3.45 3.45) (end 3.45 -3.45) (stroke (width 0.05) (type solid)) (layer "F.CrtYd"))
-    (pad "1" thru_hole circle (at 0 0 0) (size 6.4 6.4) (drill 3.2) (layers "*.Cu" "*.Mask") (solder_mask_margin 0.05))
+    (fp_rect (start -2.45 2.45) (end 2.45 -2.45) (stroke (width 0.05) (type solid)) (layer "F.CrtYd"))
+    (pad "1" thru_hole circle (at 0 0 0) (size 4.4 4.4) (drill 2.2) (layers "*.Cu" "*.Mask") (solder_mask_margin 0.05))
   )
-  (footprint "MountingHole_3.2mm_M3_Pad" (layer "F.Cu") (at 123.257 180.743 0)
-    (descr "Mounting hole for M3, plated")
-    (tags "mounting hole M3")
+  (footprint "MountingHole_2.2mm_M2_Pad" (layer "F.Cu") (at 124.257 179.743 0)
+    (descr "Mounting hole for M2, plated")
+    (tags "mounting hole M2")
     (property "Reference" "H3" (at 0 0 0) (layer "F.Fab") (hide yes) (effects (font (size 1 1))))
-    (property "Value" "MountingHole_3.2mm_M3_Pad" (at 0 0 0) (layer "F.Fab") (hide yes) (effects (font (size 1 1))))
+    (property "Value" "MountingHole_2.2mm_M2_Pad" (at 0 0 0) (layer "F.Fab") (hide yes) (effects (font (size 1 1))))
     (property "pcbkit" "holes/holes[2]" (at 0 0 0) (layer "F.Fab") (hide yes) (effects (font (size 1 1))))
-    (fp_rect (start -3.45 3.45) (end 3.45 -3.45) (stroke (width 0.05) (type solid)) (layer "F.CrtYd"))
-    (pad "1" thru_hole circle (at 0 0 0) (size 6.4 6.4) (drill 3.2) (layers "*.Cu" "*.Mask") (solder_mask_margin 0.05))
+    (fp_rect (start -2.45 2.45) (end 2.45 -2.45) (stroke (width 0.05) (type solid)) (layer "F.CrtYd"))
+    (pad "1" thru_hole circle (at 0 0 0) (size 4.4 4.4) (drill 2.2) (layers "*.Cu" "*.Mask") (solder_mask_margin 0.05))
   )
-  (footprint "MountingHole_3.2mm_M3_Pad" (layer "F.Cu") (at 103.743 180.743 0)
-    (descr "Mounting hole for M3, plated")
-    (tags "mounting hole M3")
+  (footprint "MountingHole_2.2mm_M2_Pad" (layer "F.Cu") (at 102.743 179.743 0)
+    (descr "Mounting hole for M2, plated")
+    (tags "mounting hole M2")
     (property "Reference" "H4" (at 0 0 0) (layer "F.Fab") (hide yes) (effects (font (size 1 1))))
-    (property "Value" "MountingHole_3.2mm_M3_Pad" (at 0 0 0) (layer "F.Fab") (hide yes) (effects (font (size 1 1))))
+    (property "Value" "MountingHole_2.2mm_M2_Pad" (at 0 0 0) (layer "F.Fab") (hide yes) (effects (font (size 1 1))))
     (property "pcbkit" "holes/holes[3]" (at 0 0 0) (layer "F.Fab") (hide yes) (effects (font (size 1 1))))
-    (fp_rect (start -3.45 3.45) (end 3.45 -3.45) (stroke (width 0.05) (type solid)) (layer "F.CrtYd"))
-    (pad "1" thru_hole circle (at 0 0 0) (size 6.4 6.4) (drill 3.2) (layers "*.Cu" "*.Mask") (solder_mask_margin 0.05))
+    (fp_rect (start -2.45 2.45) (end 2.45 -2.45) (stroke (width 0.05) (type solid)) (layer "F.CrtYd"))
+    (pad "1" thru_hole circle (at 0 0 0) (size 4.4 4.4) (drill 2.2) (layers "*.Cu" "*.Mask") (solder_mask_margin 0.05))
   )
   (footprint "PinHeader_1x02_P2.54mm_Vertical" (layer "F.Cu") (at 116.75 187.75 180)
     (descr "Through-hole straight pin header, 1x2, 2.54 mm pitch")
     (tags "THT pin header")
-    (property "Reference" "J1" (at 0 -3.49 180) (layer "F.SilkS") (effects (font (size 1 1) (thickness 0.15))))
+    (property "Reference" "J1" (at 0 -3.515 180) (layer "F.SilkS") (effects (font (size 1 1) (thickness 0.15))))
     (property "Value" "PinHeader_1x02_P2.54mm_Vertical" (at 0 0 0) (layer "F.Fab") (hide yes) (effects (font (size 1 1))))
     (property "LCSC Part #" "C358684" (at 0 0 0) (layer "F.Fab") (hide yes) (effects (font (size 1 1))))
@@
     (descr "Chip resistor 0603 (1608 metric), IPC-7351B nominal density")
     (tags "chip 0603 1608Metric")
-    (property "Reference" "R2" (at 0 -1.43 270) (layer "F.SilkS") (effects (font (size 1 1) (thickness 0.15))))
+    (property "Reference" "R2" (at 0 -1.455 270) (layer "F.SilkS") (effects (font (size 1 1) (thickness 0.15))))
     (property "Value" "10kohm" (at 0 0 0) (layer "F.Fab") (hide yes) (effects (font (size 1 1))))
     (property "LCSC Part #" "C25804" (at 0 0 0) (layer "F.Fab") (hide yes) (effects (font (size 1 1))))
@@
     (descr "Chip resistor 0603 (1608 metric), IPC-7351B nominal density")
     (tags "chip 0603 1608Metric")
-    (property "Reference" "R3" (at 0 -1.43 180) (layer "F.SilkS") (effects (font (size 1 1) (thickness 0.15))))
+    (property "Reference" "R3" (at 0 -1.455 180) (layer "F.SilkS") (effects (font (size 1 1) (thickness 0.15))))
     (property "Value" "330ohm" (at 0 0 0) (layer "F.Fab") (hide yes) (effects (font (size 1 1))))
     (property "LCSC Part #" "C23138" (at 0 0 0) (layer "F.Fab") (hide yes) (effects (font (size 1 1))))
