File: examples/led-bar/led-bar.kicad_pcb (KiCad board)
At the start: 2 copper layers, 55 x 18 mm, 19 parts

Commit message: p4-touch-7, blinker, led-bar: parts chosen from JLCPCB's catalogue, the fab files export
Since the parts selection buys from JLCPCB's own catalogue, these boards' support capacitors and
connectors had no orderable part and export.run refused them. parts.select chose every group
(p4-touch-7's 40 MHz crystal pinned as on the 7B board, C426988); copper unchanged.

Claude-Session: https://claude.ai/code/session_01GffCzZXi9ShujPbky1eccg
Parts:
- U1: value (none) -> SN74HC595DR

Commit message: examples: led-bar and robot-controller pass KiCad 10's starved-thermal check
PCBKit's check now counts thermal spokes as KiCad 10's DRC does, and both boards
failed it (KiCad's own DRC with refill agreed).

- led-bar: J1.5 (GND) joined the B.Cu pour through an island that joined nothing
  else (KiCad: 3 spokes to an isolated island), left by the old routing with four
  dangling GND stubs. Routed anew with today's PCBKit (design.run all): complete,
  the stubs gone; pcbkit check and kicad-cli 10 DRC (refill) clean.
- robot-controller: U1's exposed pad and its nine thermal vias (pad 17) were
  starved (11 by PCBKit, 8 by KiCad). The old import had dropped three things of
  the author's board: its minimum of 1 spoke (min_resolved_spokes 1 in the
  original project), the solid zone connection of the exposed pads (zone_connect
  2) and the tented vias. All three restored as the original has them (today's
  import keeps them); copper unchanged, pours refilled. pcbkit check and KiCad
  DRC (refill) clean; the original board with its own rules is clean in KiCad too.

Claude-Session: https://claude.ai/code/session_018URVYF1YPgyrMNetY9yT1T
Parts:
- J1: value (none) -> PinHeader_1x05_P2.54mm_Vertical
- moved C1 1.25 mm to (119.2, 191.8), turned to 0 degrees
Connections:
- R1 pad 1: Q0 -> leds[1]/anode
- R1 pad 2: leds[1]/anode -> Q0
- R2 pad 1: Q1 -> leds[2]/anode
- R2 pad 2: leds[2]/anode -> Q1
- R3 pad 1: Q2 -> leds[3]/anode
- R3 pad 2: leds[3]/anode -> Q2
- R4 pad 1: Q3 -> leds[4]/anode
- R4 pad 2: leds[4]/anode -> Q3
- R5 pad 1: Q4 -> leds[5]/anode
- R5 pad 2: leds[5]/anode -> Q4
- R6 pad 1: Q5 -> leds[6]/anode
- R6 pad 2: leds[6]/anode -> Q5
- R7 pad 1: Q6 -> leds[7]/anode
- R7 pad 2: leds[7]/anode -> Q6
- R8 pad 1: Q7 -> leds[8]/anode
- R8 pad 2: leds[8]/anode -> Q7
Routing:
- net GND: track 78.6 -> 39.1 mm, vias 0 -> 6
- net Q7: track 59.4 -> 47.9 mm
- net Q6: track 55.1 -> 51.4 mm
- net Q2: track 28.9 -> 25.8 mm
- net Q4: track 42.1 -> 39.3 mm
- net +5V: track 25.6 -> 23.6 mm
- net leds[6]/anode: track 7.98 -> 6.18 mm
- net leds[7]/anode: track 7.81 -> 6.18 mm
- net leds[5]/anode: track 7.68 -> 6.11 mm
- net leds[1]/anode: track 7.72 -> 6.18 mm
- net leds[4]/anode: track 7.72 -> 6.18 mm
- net leds[8]/anode: track 7.67 -> 6.18 mm
- net leds[3]/anode: track 7.66 -> 6.18 mm
- net leds[2]/anode: track 7.65 -> 6.18 mm
- net Q5: track 46.3 -> 45.1 mm
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