File: retro/delta-s02/Delta-S02.kicad_pcb (KiCad board)
At the start: 2 copper layers, 285.5 x 150.2 mm, 186 parts

Commit message: Boards pass check and KiCad 10's DRC again: holes in courtyards, the USB net rename
pcbkit's check now has KiCad 10's pth/npth_inside_courtyard (pcbkit be5b6955), and 13 boards
failed it. KiCad's own DRC (kicad-cli 10) reports the same holes on every one of them.

- Parts that really stand above the holes under them (a screen or a Nano on its sockets, the
  Delta-S02's КМ-6 capacitors flat under its chips, as the factory placed them): a courtyard rule
  for the pair, written to each board's .kicad_dru, so KiCad's DRC agrees.
- Real collisions moved: servo-controller's dial 3 mm up (the Nano's socket pins came out under
  it), c3-pocket's fourth M3 hole from under a cell holder to the top edge's middle, s3-rgb's
  D-pad 2 mm up (a holder's peg came through under the down key).
- v003-emu, c3-pocket, rp2040-tft, rp2350-psram, s3-rgb, teensy41: re-routed for the standard USB
  block's renamed net (usb/raw is usb/vbusIn since pcbkit 2088839e): their tracks still carried
  the old name and shorted the fuse and connector pads.
- p4-touch-7: its board file still had a courtyard for the panel the design gives none (KiCad
  reported 114 courtyard errors); written again.

Measured on the dev host: all 44 registry boards `pcbkit check` complete with 0 errors, and
kicad-cli pcb drc 0 errors on every board.

Claude-Session: https://claude.ai/code/session_018URVYF1YPgyrMNetY9yT1T
Routing:
- net KC: track 60.1 -> 56.8 mm
- net nBK: track 110.8 -> 108.0 mm
- net RWE: track 118.8 -> 116.2 mm
- net KSEL: track 58.9 -> 56.3 mm
- net RAS: track 194.0 -> 192.1 mm
- net M6: track 214.4 -> 212.5 mm
- net PA14: track 38.8 -> 37.0 mm
- net RA7: track 122.6 -> 120.8 mm
- net nIORQ: track 183.1 -> 181.3 mm
- net M9: track 46.5 -> 44.8 mm
- net RA1: track 124.8 -> 123.0 mm
- net MD3: track 140.1 -> 138.3 mm
- net KL1: track 84.4 -> 82.7 mm
- net A5: track 227.6 -> 225.9 mm
- net V5: track 148.8 -> 147.2 mm
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
Commit message: registry: every board rebuilt with pcbkit main 4684674e6 - the bought part named on the board
pcbkit dc07fdfd6 writes the bought row's MPN and Manufacturer (the design's own kept as DesignMPN /
DesignManufacturer) and the build chooses parts before it places (6361ec104). Each of the 44 boards
was rebuilt (; the two P4 boards  only: their builds reroute pairs):
copper unchanged on all 44 (segments, arcs and vias counted before and after), placement kept; the
Arduino and lab boards now carry the parts the catalogue gives them. The check gains only the new
judgements: part-maker (a part bought from another maker) and part-missing on hand-fitted modules
(DS1 sockets); p4-touch-7 loses part-stale. The P4 boards keep their hole-clearance errors (a
reroute is Team 3's).

Claude-Session: https://claude.ai/code/session_01BAgp959tApA8aEg85EYgfb
Other:
- copper layers 2 -> 4

Commit message: retro/delta-s02: back on the 2 copper layers it was routed on, rebuilt with pcbkit main aa82f6c3b
e65077e's rebuild (pcbkit 4684674e6, before 781a3d329) raised the recorded stack to the 4 layers the
plan estimates, so the board file, the model and its fab archive said 4 while every track is on F/B
(order-archive true, web-test 'every demo board opens complete'). Rebuilt from the 2-layer board of
580e1af with main (pcbkit route): 2 copper layers, 1.51 mm core, 7924 segments as before, check
complete (2 part-missing warnings on the hand-fitted parts, as before); min_hole_to_hole 0.2 (main's
hole spacing); two parts re-chosen from today's catalogue (C 300 pF C376827, R 1.3 kohm C25988).

Claude-Session: https://claude.ai/code/session_01BAgp959tApA8aEg85EYgfb
Other:
- copper layers 4 -> 2
Changed lines of the file:
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@@
   (layers
     (0 "F.Cu" signal)
-    (1 "In1.Cu" signal)
-    (2 "In2.Cu" signal)
     (31 "B.Cu" signal)
     (32 "B.Adhes" user "B.Adhesive") (33 "F.Adhes" user "F.Adhesive") (34 "B.Paste" user) (35 "F.Paste" user)
@@
       (layer "F.Mask" (type "Top Solder Mask") (color "Green") (thickness 0.01))
       (layer "F.Cu" (type "copper") (thickness 0.035))
-      (layer "dielectric 1" (type "core") (thickness 0.203) (material "FR4"))
-      (layer "In1.Cu" (type "copper") (thickness 0.035))
-      (layer "dielectric 2" (type "prepreg") (thickness 1.03) (material "FR4"))
-      (layer "In2.Cu" (type "copper") (thickness 0.035))
-      (layer "dielectric 3" (type "core") (thickness 0.203) (material "FR4"))
+      (layer "dielectric 1" (type "core") (thickness 1.51) (material "FR4"))
       (layer "B.Cu" (type "copper") (thickness 0.035))
       (layer "B.Mask" (type "Bottom Solder Mask") (color "Green") (thickness 0.01))
@@
     (property "Reference" "C2" (at 0 0 0) (layer "F.Fab") (hide yes) (effects (font (size 1 1))))
     (property "Value" "300pF" (at 0 0 0) (layer "F.Fab") (hide yes) (effects (font (size 1 1))))
-    (property "LCSC Part #" "C49326637" (at 0 0 0) (layer "F.Fab") (hide yes) (effects (font (size 1 1))))
-    (property "MPN" "0603X7R301K500NT" (at 0 0 0) (layer "F.Fab") (hide yes) (effects (font (size 1 1))))
-    (property "Manufacturer" "AIDE(爱迪电容)" (at 0 0 0) (layer "F.Fab") (hide yes) (effects (font (size 1 1))))
+    (property "LCSC Part #" "C376827" (at 0 0 0) (layer "F.Fab") (hide yes) (effects (font (size 1 1))))
+    (property "MPN" "TCC0603X7R301K500CT" (at 0 0 0) (layer "F.Fab") (hide yes) (effects (font (size 1 1))))
+    (property "Manufacturer" "CCTC" (at 0 0 0) (layer "F.Fab") (hide yes) (effects (font (size 1 1))))
     (property "pcbkit" "C2" (at 0 0 0) (layer "F.Fab") (hide yes) (effects (font (size 1 1))))
     (property "pcbkit-need" "5125ccf60564 MPN Manufacturer" (at 0 0 0) (layer "F.Fab") (hide yes) (effects (font (size 1 1))))
@@
     (property "Reference" "R53" (at 0 0 0) (layer "F.Fab") (hide yes) (effects (font (size 1 1))))
     (property "Value" "1.3kohm" (at 0 0 0) (layer "F.Fab") (hide yes) (effects (font (size 1 1))))
-    (property "LCSC Part #" "C365102" (at 0 0 0) (layer "F.Fab") (hide yes) (effects (font (size 1 1))))
-    (property "MPN" "HPCR0603F1K30K9" (at 0 0 0) (layer "F.Fab") (hide yes) (effects (font (size 1 1))))
-    (property "Manufacturer" "RESI" (at 0 0 0) (layer "F.Fab") (hide yes) (effects (font (size 1 1))))
+    (property "LCSC Part #" "C25988" (at 0 0 0) (layer "F.Fab") (hide yes) (effects (font (size 1 1))))
+    (property "MPN" "0603WAJ0132T5E" (at 0 0 0) (layer "F.Fab") (hide yes) (effects (font (size 1 1))))
+    (property "Manufacturer" "UNI-ROYAL(Uniroyal Elec)" (at 0 0 0) (layer "F.Fab") (hide yes) (effects (font (size 1 1))))
     (property "pcbkit" "R53" (at 0 0 0) (layer "F.Fab") (hide yes) (effects (font (size 1 1))))
     (property "pcbkit-need" "234e4b7105fa MPN Manufacturer" (at 0 0 0) (layer "F.Fab") (hide yes) (effects (font (size 1 1))))
